File: 5_Way_Flex_Switch/5_Way_Flex_Switch.sch (EAGLE design)
At the start: 9 parts

Commit message: Licenses
Parts:
- removed MOD1: CONFIGURATION_BRD, CYCFI_Module_castellated:CONFIGURATION_BRD
- added CB1: CONFIGURATION_BRD_PADS, CYCFI_Module_castellated:CONFIGURATION_BRD_PADS
Connections:
- removed net M1: MOD1.M, U$1.M1
- removed net N2: MOD1.N2, U$1.N2
- new net N$13: CB1.M1, U$1.M1
- new net N$15: CB1.N2, U$1.N2
- new net N$16: CB1.M2, U$1.M2
- new net N$17: CB1.B2, U$1.B2
- new net N$2: CB1.COM2, U$1.COM2
- new net N$3: CB1.COM1, U$1.COM1
- net 1-IC: now also CB1.1-IC; no longer MOD1.1-IC
- net 1-OC: now also CB1.1-OC; no longer MOD1.1-OC
- net 2-IC: now also CB1.2-IC; no longer MOD1.2-IC
- net 2-OC: now also CB1.2-OC; no longer MOD1.2-OC
- net 3-IC: now also CB1.3-IC; no longer MOD1.3-IC
- net 3-OC: now also CB1.3-OC; no longer MOD1.3-OC
- net 4-IC: now also CB1.4-IC; no longer MOD1.4-IC
- net 4-OC: now also CB1.4-OC; no longer MOD1.4-OC
- net B1: now also CB1.B1; no longer MOD1.B
- net GND: now also CB1.GND, CB1.GND1; no longer MOD1.GND
- net IN+: now also CB1.OUT-; no longer U$1.COM1
- net IN-: now also CB1.OUT+; no longer MOD1.IN-, U$1.COM2
- net N1: now also CB1.N1; no longer MOD1.N
Other:
- note added: "-(SW)"
- note added: "20160601"
- note added: "5 Way Flex Switch Projecy by Cycfi Research is licensed under a Creative Commons Attribution-ShareAlike 4.0 International License. Copyright CYCFI Research Inc. 2013-2016"
- note added: "ACTIVE VOLUME INPUT SIGNAL"
- note added: "ACTIVE VOLUME PWR"
- note added: "B1"
- note added: "B2"
- note added: "BATT"
- note added: "BLEND CONTROL"
- note added: "COM1"
- note added: "COM2"
- note added: "GND(-)"
- note added: "IC(C-)"
- note added: "M1"
- note added: "M2"
- note added: "N1"
- note added: "N2"
- note added: "NOTES: *OC(C+) = Outer coil terminal *IC(C-) = Inner coil terminal"
- note added: "OC(C+)"
- note added: "PASSIVE PICKUP INPUTS"
- note added: "PU1-IC(C-)"
- note added: "PU1-OC(C+)"
- note added: "PU2-IC(C-)"
- note added: "PU2-OC(C+)"
- note added: "PU3-IC(C-)"
- note added: "PU3-OC(C+)"
- note added: "PU4-IC(C-)"
- note added: "PU4-OC(C+)"
- note added: "VCC(+)"
- note added: "v1.2"
- note removed: "5 Way Flex Switch Project by Cycfi Research is licensed under a Creative Commons Attribution-NonCommercial 4.0 International License. http://creativecommons.org/licenses/by-nc/4.0/ Copyright CYCFI Research Inc. 2013-2016"
- note removed: "ACTIVE VOL PWR"
- note removed: "BLEND"
- note removed: "CONFIGURATION BOARD"
- note removed: "GND"
- note removed: "IC"
- note removed: "NOTES: *OC = Outer coil terminal *IC = Inner coil terminal"
- note removed: "OC"
- note removed: "PU1-IC"
- note removed: "PU1-OC"
- note removed: "PU2-IC\"
- note removed: "PU2-OC"
- note removed: "PU3-IC"
- note removed: "PU3-OC"
- note removed: "PU4-IC"
- note removed: "PU4-OC"
- note removed: "SW"
- note removed: "VCC"
