File: XR_Controls/Blend_Control/Blend_Control.sch (EAGLE design)
At the start: 4 parts

Commit message: Licenses
Other:
- note added: "Blend Control Project by Cycfi Research is licensed under a Creative Commons Attribution-ShareAlike 4.0 International License. Copyright CYCFI Research Inc. 2013-2016"
- note removed: "XR Controls Project by Cycfi Research is licensed under a Creative Commons Attribution-NonCommercial 4.0 International License. http://creativecommons.org/licenses/by-nc/4.0/ Copyright CYCFI Research Inc. 2013-2016"
Changed lines of the file:
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@@
 <text x="177.8" y="19.05" size="2.54" layer="95">Blend Control</text>
 <text x="253.365" y="6.985" size="2.1844" layer="95">v1.46</text>
-<text x="7.62" y="12.7" size="2.54" layer="95">XR Controls Project by Cycfi Research is licensed under a
-Creative Commons Attribution-NonCommercial 4.0 International License.
-http://creativecommons.org/licenses/by-nc/4.0/
+<text x="7.62" y="12.7" size="2.54" layer="95">Blend Control Project by Cycfi Research is licensed under a
+Creative Commons Attribution-ShareAlike 4.0 International License.
 Copyright CYCFI Research Inc. 2013-2016</text>
 <text x="200.66" y="11.43" size="2.54" layer="95">2016040</text>
