File: Active_Volume/Active_Volume.sch (EAGLE design)
At the start: 10 parts, among them U1 XR_PREAMP

Commit message: Licenses
Other:
- note added: "-(SW)"
- note added: "Active Volume Project by Cycfi Research is licensed under a Creative Commons Attribution-ShareAlike 4.0 International License. Copyright CYCFI Research Inc. 2013-2016"
- note added: "COIL"
- note added: "GND(-)"
- note added: "OUTPUT JACK"
- note added: "PWR"
- note added: "TONE CONTROL"
- note added: "VCC(+)"
- note removed: "Active Volume Project by Cycfi Research is licensed under a Creative Commons Attribution-NonCommercial 4.0 International License. http://creativecommons.org/licenses/by-nc/4.0/ Copyright CYCFI Research Inc. 2013-2016"
- note removed: "GND"
- note removed: "IN+"
- note removed: "IN-"
- note removed: "INPUT"
- note removed: "OUTPUT"
- note removed: "TONE"
- note removed: "VCC"
- note removed: "VOL PWR"
- moved on the sheet: H1

Commit message: *organize 5-waay switch and its configuration board(a and b) *update license date *remove red frame schem pdf files, change with black frame *update document number
Other:
- note added: "201705"
- note added: "201706"
- note added: "Active Volume Project by Cycfi Research is licensed under a Creative Commons Attribution-ShareAlike 4.0 International License. Copyright CYCFI Research Inc. 2013-2017"
- note removed: "2016039"
- note removed: "Active Volume Project by Cycfi Research is licensed under a Creative Commons Attribution-ShareAlike 4.0 International License. Copyright CYCFI Research Inc. 2013-2016"
Changed lines of the file:
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@@
 <text x="177.8" y="19.05" size="2.54" layer="95">Active Volume</text>
 <text x="252.73" y="6.985" size="2.1844" layer="95">v1.1</text>
-<text x="7.62" y="12.7" size="2.54" layer="95">Active Volume Project by Cycfi Research is licensed under a
+<text x="17.78" y="12.7" size="3.048" layer="95">Active Volume Project by Cycfi Research is licensed under a
 Creative Commons Attribution-ShareAlike 4.0 International License.
-Copyright CYCFI Research Inc. 2013-2016</text>
-<text x="200.66" y="11.43" size="2.54" layer="95">2016039</text>
+Copyright CYCFI Research Inc. 2013-2017</text>
+<text x="200.66" y="11.43" size="2.54" layer="95">201705</text>
 <wire x1="192.47528125" y1="25.047221875" x2="190.115640625" y2="25.047221875" width="0" layer="94"/>
 <wire x1="190.115640625" y1="25.047221875" x2="188.10833125" y2="25.047225" width="0" layer="94"/>
@@
 <instance part="SUPPLY4" gate="GND" x="105.41" y="88.9"/>
 <instance part="P+3" gate="VCC" x="105.41" y="151.13" smashed="yes">
-<attribute name="VALUE" x="106.68" y="149.86" size="1.778" layer="96"/>
+<attribute name="VALUE" x="104.14" y="152.4" size="1.778" layer="96"/>
 </instance>
 <instance part="FRAME1" gate="G$1" x="0" y="0"/>
@@
 <text x="177.8" y="19.05" size="2.54" layer="95">Active Volume</text>
 <text x="252.73" y="6.985" size="2.1844" layer="95">v1.1</text>
-<text x="7.62" y="12.7" size="2.54" layer="95">Active Volume Project by Cycfi Research is licensed under a
+<text x="22.86" y="12.7" size="3.048" layer="95">Active Volume Project by Cycfi Research is licensed under a
 Creative Commons Attribution-ShareAlike 4.0 International License.
-Copyright CYCFI Research Inc. 2013-2016</text>
-<text x="200.66" y="11.43" size="2.54" layer="95">2016039</text>
+Copyright CYCFI Research Inc. 2013-2017</text>
+<text x="200.66" y="11.43" size="2.54" layer="95">201706</text>
 <wire x1="192.47528125" y1="25.047221875" x2="190.115640625" y2="25.047221875" width="0" layer="94"/>
 <wire x1="190.115640625" y1="25.047221875" x2="188.10833125" y2="25.047225" width="0" layer="94"/>
