File: XR_Preamp/Version_1_5/XR_Preamp.sch (EAGLE design)
At the start: 9 parts

Commit message: Added Preamp V 1.5
Parts:
- removed H1: MA02-1, con-lstb:MA02-1
- removed H2: (no value), con-lstb:MA04-2
- removed H3: 3PIN-SMD-2.54MM, CYCFI_Con:3PIN-SMD-2.54MM
- removed H4, H5: (no value), con-lstb:MA06-1EDITED
- removed MOD1: CONFIGURATION_BRD, CYCFI_Module_castellated:CONFIGURATION_BRD
- removed U$1: 5WAY_SW_CASTELLATED, CYCFI_switch:5WAY_SW_CASTELLATED
- added C3: 4.7uF, resistor:C-EUC0603
- added C4: 0.1uf, resistor:C-EUC0402
- added C5: 4.7uF, resistor:C-EUC0402
- added PAD1, PAD2, PAD3, PAD4, PAD5: WIREPAD2,15/1,0, wirepad:1,6/0,8
- added R1: 200K, resistor:R-EU_R0402
- added R2: 27K, resistor:R-EU_R0402
- added R3: 22K, resistor:R-EU_R0402
- added R4, R5: 10K, resistor:R-EU_R0402
- added R6: 4.7K, resistor:R-EU_R0402
- added R7: 1K, resistor:R-EU_R0402
- added T1, T2: 2SC3324, transistor:BC846
- C2: value 0.1uF -> 100pF; device resistor:C-EUC0603 -> resistor:C-EUC0402
Connections:
- removed net 1-IC: H4.3, MOD1.1-IC
- removed net 1-OC: H4.1, MOD1.1-OC
- removed net 2-IC: H4.6, MOD1.2-IC
- removed net 2-OC: H4.4, MOD1.2-OC
- removed net 3-IC: H5.3, MOD1.3-IC
- removed net 3-OC: H5.1, MOD1.3-OC
- removed net 4-IC: H5.6, MOD1.4-IC
- removed net 4-OC: H5.4, MOD1.4-OC
- removed net B1: H2.4, MOD1.B, U$1.B1
- removed net IN+: H2.7, U$1.COM1
- removed net IN-: H2.8, MOD1.IN-, U$1.COM2
- removed net M1: MOD1.M, U$1.M1
- removed net N1: H2.2, MOD1.N, U$1.N1
- removed net N2: MOD1.N2, U$1.N2
- removed net SW: H1.1, H2.1
- removed net VBATT: C1.1, C2.1, H1.2, H3.1
- new net GAIN: PAD1.P, R7.2, T1.E
- new net IN: C1.1, C2.2, PAD3.P
- new net N$1: C1.2, R1.1, R2.2, T1.B
- new net N$3: C5.2, R4.2, T2.E
- new net OUT: PAD5.P, R6.2
- new net OUT1: C5.1, R5.2, R6.1
- new net VCVF: R1.2, R3.1, T1.C, T2.B
- net GND: now also C2.1, C3.1, C4.1, PAD2.P, R2.1, R4.1, R5.1, R7.1; no longer C1.2, C2.2, H2.5, H2.6, H3.3, H4.2, H4.5, H5.2, H5.5, MOD1.GND
- net VCC: now also C3.2, C4.2, PAD4.P, R3.2, T2.C; no longer H2.3, H3.2
Other:
- note added: "1"
- note added: "1/2"
- note added: "2"
- note added: "2/2"
- note added: "2016008"
- note added: "3"
- note added: "CASTELLATED PADS"
- note added: "GND"
- note added: "NOTE: *Gain Adjustment Trimmer"
- note added: "TR1 500 0hms"
- note added: "VCC"
- note added: "XR Preamp"
- note added: "XR Preamp Project by Cycfi Research is licensed under a Creative Commons Attribution-NonCommercial 4.0 International License. http://creativecommons.org/licenses/by-nc/4.0/ Copyright CYCFI Research Inc. 2013-2016"
- note added: "v1.5"
- note removed: "-(SW)"
- note removed: "2016037"
- note removed: "5 Way Flex Switch"
- note removed: "5 Way Flex Switch Project by Cycfi Research is licensed under a Creative Commons Attribution-NonCommercial 4.0 International License. http://creativecommons.org/licenses/by-nc/4.0/ Copyright CYCFI Research Inc. 2013-2016"
- note removed: "ACTIVE VOLUME INPUT SIGNAL"
- note removed: "ACTIVE VOLUME PWR"
- note removed: "BATT"
- note removed: "BLEND CONTROL"
- note removed: "CONFIGURATION BOARD"
- note removed: "GND(-)"
- note removed: "H1"
- note removed: "IC(C-)"
- note removed: "NOTES: *OC(C+) = Outer coil terminal *IC(C-) = Inner coil terminal"
- note removed: "OC(C+)"
- note removed: "OUT+"
- note removed: "OUT-"
- note removed: "OUTPUT HEADERS"
- note removed: "PASSIVE PICKUP INPUTS"
- note removed: "PU1"
- note removed: "PU1-IC(C-)"
- note removed: "PU1-OC(C+)"
- note removed: "PU2"
- note removed: "PU2-IC(C-)"
- note removed: "PU2-OC(C+)"
- note removed: "PU3"
- note removed: "PU3-IC(C-)"
- note removed: "PU3-OC(C+)"
- note removed: "PU4"
- note removed: "PU4-IC(C-)"
- note removed: "PU4-OC(C+)"
- note removed: "PWR SWITCH"
- note removed: "STRING GND"
- note removed: "VBATT"
- note removed: "VCC(+)"
- note removed: "v1.1"

Commit message: Licenses
Other:
- note added: "XR Preamp Project by Cycfi Research is licensed under a Creative Commons Attribution-ShareAlike 4.0 International License. Copyright CYCFI Research Inc. 2013-2016"
- note removed: "XR Preamp Project by Cycfi Research is licensed under a Creative Commons Attribution-NonCommercial 4.0 International License. http://creativecommons.org/licenses/by-nc/4.0/ Copyright CYCFI Research Inc. 2013-2016"
Changed lines of the file:
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@@
 <text x="252.73" y="6.985" size="2.1844" layer="95">v1.5</text>
 <text x="7.62" y="12.7" size="2.54" layer="95">XR Preamp Project by Cycfi Research is licensed under a
-Creative Commons Attribution-NonCommercial 4.0 International License.
-http://creativecommons.org/licenses/by-nc/4.0/
+Creative Commons Attribution-ShareAlike 4.0 International License.
 Copyright CYCFI Research Inc. 2013-2016</text>
 <text x="200.66" y="11.43" size="2.54" layer="95">2016008</text>
@@
 <text x="252.73" y="6.985" size="2.1844" layer="95">v1.5</text>
 <text x="7.62" y="12.7" size="2.54" layer="95">XR Preamp Project by Cycfi Research is licensed under a
-Creative Commons Attribution-NonCommercial 4.0 International License.
-http://creativecommons.org/licenses/by-nc/4.0/
+Creative Commons Attribution-ShareAlike 4.0 International License.
 Copyright CYCFI Research Inc. 2013-2016</text>
 <text x="200.66" y="11.43" size="2.54" layer="95">2016008</text>

Commit message: *organize 5-waay switch and its configuration board(a and b) *update license date *remove red frame schem pdf files, change with black frame *update document number
Other:
- note added: "201715"
- note added: "201716"
- note added: "XR Preamp Project by Cycfi Research is licensed under a Creative Commons Attribution-ShareAlike 4.0 International License. Copyright CYCFI Research Inc. 2013-2017"
- note removed: "2016008"
- note removed: "XR Preamp Project by Cycfi Research is licensed under a Creative Commons Attribution-ShareAlike 4.0 International License. Copyright CYCFI Research Inc. 2013-2016"
Changed lines of the file:
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@@
 <text x="7.62" y="12.7" size="2.54" layer="95">XR Preamp Project by Cycfi Research is licensed under a
 Creative Commons Attribution-ShareAlike 4.0 International License.
-Copyright CYCFI Research Inc. 2013-2016</text>
-<text x="200.66" y="11.43" size="2.54" layer="95">2016008</text>
+Copyright CYCFI Research Inc. 2013-2017</text>
+<text x="200.66" y="11.43" size="2.54" layer="95">201716</text>
 <wire x1="192.47528125" y1="25.047221875" x2="190.115640625" y2="25.047221875" width="0" layer="94"/>
 <wire x1="190.115640625" y1="25.047221875" x2="188.10833125" y2="25.047225" width="0" layer="94"/>
@@
 <text x="7.62" y="12.7" size="2.54" layer="95">XR Preamp Project by Cycfi Research is licensed under a
 Creative Commons Attribution-ShareAlike 4.0 International License.
-Copyright CYCFI Research Inc. 2013-2016</text>
-<text x="200.66" y="11.43" size="2.54" layer="95">2016008</text>
+Copyright CYCFI Research Inc. 2013-2017</text>
+<text x="200.66" y="11.43" size="2.54" layer="95">201715</text>
 <wire x1="192.47528125" y1="25.047221875" x2="190.115640625" y2="25.047221875" width="0" layer="94"/>
 <wire x1="190.115640625" y1="25.047221875" x2="188.10833125" y2="25.047225" width="0" layer="94"/>
