File: Active_Volume_Preamp/Active_Volume_Preamp.sch (EAGLE design)
At the start: 19 parts, among them T1 2SC3324, T2 2SC3324

Commit message: Updated BOM and Document Number
Parts:
- removed C1, C3: 4.7uF, resistor:C-EUC0603
- removed C2: 100pF, resistor:C-EUC0402
- removed C4: 0.1uf, resistor:C-EUC0402
- removed C5: 4.7uF, resistor:C-EUC0402
- removed R1: 200K, resistor:R-EU_R0402
- removed R2: 27K, resistor:R-EU_R0402
- removed R3: 22K, resistor:R-EU_R0402
- removed R4, R5: 10K, resistor:R-EU_R0402
- removed R6: 4.7K, resistor:R-EU_R0402
- removed R7: 1K, resistor:R-EU_R0402
- removed T1, T2: 2SC3324, transistor:BC846
- added H1: (no value), con-lstb:MA07-2
- added PAD6, PAD7: (no value), wirepad:SMD2
- added TR1: TC33X-2-201E, CYCFI_Passive:TC33X-2-201E
- added U1: XR_PREAMP, CYCFI_Module_castellated:XR_PREAMP
- PAD1, PAD2, PAD3, PAD4, PAD5: value WIREPAD2,15/1,0 -> (none); device wirepad:1,6/0,8 -> wirepad:SMD2
Connections:
- removed net GAIN: PAD1.P, R7.2, T1.E
- removed net IN: C1.1, C2.2, PAD3.P
- removed net N$3: C5.2, R4.2, T2.E
- removed net OUT: PAD5.P, R6.2
- removed net OUT1: C5.1, R5.2, R6.1
- removed net VCVF: R1.2, R3.1, T1.C, T2.B
- new net INPUT: H1.5, U1.IN
- new net OUT(PREAMP): H1.8, U1.OUT
- new net OUT(SEL): H1.10, PAD2.P
- new net OUT(VOL): H1.1, H1.4, PAD3.P
- new net SW: H1.2, H1.9
- net GND: now also H1.13, H1.14, H1.3, H1.6, H1.7, PAD1.P, PAD4.P, PAD5.P, PAD6.P, PAD7.P, TR1.3, U1.GND; no longer C2.1, C3.1, C4.1, PAD2.P, R2.1, R4.1, R5.1, R7.1
- net N$1: now also TR1.2, U1.GAIN; no longer C1.2, R1.1, R2.2, T1.B
- net VCC: now also H1.11, H1.12, U1.VCC; no longer C3.2, C4.2, PAD4.P, R3.2, T2.C
Other:
- note added: "-(SW)"
- note added: "2016039"
- note added: "500 ohms"
- note added: "Active Volume"
- note added: "Active Volume for XR Project by Cycfi Research is licensed under a Creative Commons Attribution-ShareAlike 4.0 International License. http://creativecommons.org/licenses/by-sa/4.0/ Copyright CYCFI Research Inc. 2013-2017"
- note added: "COIL"
- note added: "GND(-)"
- note added: "IN"
- note added: "INSERT"
- note added: "NOTES: *POTENTIOMETER BREAKOUT = SMD pads for potentiometer breakout board (POT1)"
- note added: "OUT"
- note added: "OUTPUT HEADERS"
- note added: "OUTPUT JACK"
- note added: "OUT\"
- note added: "POT1 25K"
- note added: "POTENTIOMETER BREAKOUT"
- note added: "PWR"
- note added: "SW"
- note added: "TONE CONTROL"
- note added: "VCC(+)"
- note added: "v1.1"
- note removed: "1/2"
- note removed: "2/2"
- note removed: "2016008"
- note removed: "CASTELLATED PADS"
- note removed: "GND"
- note removed: "NOTE: *Gain Adjustment Trimmer"
- note removed: "TR1 500 0hms"
- note removed: "VCC"
- note removed: "XR Preamp"
- note removed: "XR Preamp Project by Cycfi Research is licensed under a Creative Commons Attribution-ShareAlike 4.0 International License. http://creativecommons.org/licenses/by-sa/4.0/ Copyright CYCFI Research Inc. 2013-2017"
- note removed: "v1.5"
