File: Resonant_Filter/Resonant_Filter.sch (EAGLE design)
At the start: 9 parts

Commit message: Updated BOM and Document Number
Parts:
- removed CB1: CONFIGURATION_BRD_PADS, CYCFI_Module_castellated:CONFIGURATION_BRD_PADS
- removed H3: 3PIN-SMD-2.54MM, CYCFI_Con:3PIN-SMD-2.54MM
- removed H4, H5: (no value), con-lstb:MA06-1EDITED
- removed U$1: 5WAY_SW_CASTELLATED, CYCFI_switch:5WAY_SW_CASTELLATED
- added C3: 0.1uF, resistor:C-EUC0603
- added C4: 4.7uF, resistor:C-EUC0603
- added C5: 1uF, resistor:C-EUC0805
- added C6: 100pF, resistor:C-EUC0805
- added C7, C8: 3.3nF, resistor:C-EUC0805
- added PAD1, PAD2, PAD3, PAD4, PAD5, PAD6, PAD7: (no value), wirepad:SMD2
- added PAD8: (no value), wirepad:1,6/0,9
- added POT1-A: PDB182-GTR02, CYCFI_Passive:PDB182-GTR02
- added R1: 150K, resistor:R-EU_R0402
- added R10, R11, R2, R3: 100K, resistor:R-EU_R0402
- added R4: 20K, resistor:R-EU_R0402
- added R5: 60.4K, resistor:R-EU_R0402
- added R6: 47K, resistor:R-EU_R0402
- added R7: 4.7K, resistor:R-EU_R0402
- added R8, R9: 3.3K, resistor:R-EU_R0603
- added T1: 2SC3324, transistor:BC846
- added U1: OPA209, CYCFI:OPA836
- C1: value 4.7uF -> 0.1uF
- C2: value 0.1uF -> 1uF; device resistor:C-EUC0603 -> resistor:C-EUC0805
- H1: value MA02-1 -> (none); device con-lstb:MA02-1 -> con-lstb:MA08-1
- H2: device con-lstb:MA04-2 -> con-lstb:MA04-1
Connections:
- removed net 1-IC: CB1.1-IC, H4.3
- removed net 1-OC: CB1.1-OC, H4.1
- removed net 2-IC: CB1.2-IC, H4.6
- removed net 2-OC: CB1.2-OC, H4.4
- removed net 3-IC: CB1.3-IC, H5.3
- removed net 3-OC: CB1.3-OC, H5.1
- removed net 4-IC: CB1.4-IC, H5.6
- removed net 4-OC: CB1.4-OC, H5.4
- removed net B1: CB1.B1, H2.4, U$1.B1
- removed net IN+: CB1.OUT-, H2.7
- removed net IN-: CB1.OUT+, H2.8
- removed net N$13: CB1.M1, U$1.M1
- removed net N$15: CB1.N2, U$1.N2
- removed net N$16: CB1.M2, U$1.M2
- removed net N$17: CB1.B2, U$1.B2
- removed net N1: CB1.N1, H2.2, U$1.N1
- removed net SW: H1.1, H2.1
- removed net VBATT: C1.1, C2.1, H1.2, H3.1
- removed net VCC: H2.3, H3.2
- new net 1: H1.5, R4.2, T1.E
- new net 2: C8.1, H2.3, POT1-AG$2.2, R11.2
- new net 3: H1.7, U1.+IN
- new net 4: H2.1, R8.1
- new net 5: C7.2, H2.2
- new net ASDADS: C5.1, R6.2, R7.1
- new net BYP: H1.1, PAD1.P
- new net EQ: H1.2, R7.2
- new net INPUT: C1.1, PAD2.P
- new net N$1: POT1-AG$1.3, R10.2, R8.2
- new net N$4: C1.2, R2.1, R3.2, T1.B
- new net N$8: C2.2, R5.2
- new net PA-3: PAD3.P, R1.2
- new net PTB-1: C5.2, C6.2, H1.6, PAD5.P, U1.OUT
- new net PTB-2: PAD6.P, U1.-IN
- new net PTB-3: C6.1, PAD4.P, R5.1
- new net VIN: C3.2, C4.2, H1.3, R2.2, T1.C, U1.V+
- net GND: now also C2.1, C3.1, C4.1, C8.2, H1.4, H1.8, H2.4, PAD7.P, PAD8.P, R1.1, R3.1, R4.1, R6.1, U1.V-; no longer C1.2, C2.2, CB1.GND, CB1.GND1, H2.5, H2.6, H3.3, H4.2, H4.5, H5.2, H5.5
- net N$2: now also C7.1, POT1-AG$1.2, R10.1, R9.1; no longer CB1.COM2, U$1.COM2
- net N$3: now also POT1-AG$2.3, R11.1, R9.2; no longer CB1.COM1, U$1.COM1
Other:
- note added: "+"
- note added: "-"
- note added: "1"
- note added: "2"
- note added: "201709"
- note added: "3"
- note added: "FREQ"
- note added: "FREQUENCY CONTROL"
- note added: "IN"
- note added: "INS"
- note added: "OUT"
- note added: "PADS FOR DUAL POTENTIOMETER BREAKOUT"
- note added: "POT1-A"
- note added: "POT1-A 100K"
- note added: "POT1-B"
- note added: "POT1-B 100K"
- note added: "Q CONTROL"
- note added: "Resonant Filter"
- note added: "Resonant Filter for XR Project by Cycfi Research is licensed under a Creative Commons Attribution-ShareAlike 4.0 International License. http://creativecommons.org/licenses/by-sa/4.0/ Copyright CYCFI Research Inc. 2013-2017"
- note added: "SOLDERING PAD FOR POTENTIOMETER CASE"
- note added: "v1.46"
- note removed: "-(SW)"
- note removed: "2016037"
- note removed: "5 Way Flex Switch"
- note removed: "5 Way Flex Switch for XR Project by Cycfi Research is licensed under a Creative Commons Attribution-ShareAlike 4.0 International License. http://creativecommons.org/licenses/by-sa/4.0/ Copyright CYCFI Research Inc. 2013-2017"
- note removed: "ACTIVE VOLUME INPUT SIGNAL"
- note removed: "ACTIVE VOLUME PWR"
- note removed: "B1"
- note removed: "B2"
- note removed: "BATT"
- note removed: "BLEND CONTROL"
- note removed: "COM1"
- note removed: "COM2"
- note removed: "GND(-)"
- note removed: "H1"
- note removed: "IC(C-)"
- note removed: "M1"
- note removed: "M2"
- note removed: "N1"
- note removed: "N2"
- note removed: "NOTES: *OC(C+) = Outer coil terminal *IC(C-) = Inner coil terminal"
- note removed: "OC(C+)"
- note removed: "OUT+"
- note removed: "OUT-"
- note removed: "OUTPUT HEADERS"
- note removed: "PASSIVE PICKUP INPUTS"
- note removed: "PU1"
- note removed: "PU1-IC(C-)"
- note removed: "PU1-OC(C+)"
- note removed: "PU2"
- note removed: "PU2-IC(C-)"
- note removed: "PU2-OC(C+)"
- note removed: "PU3"
- note removed: "PU3-IC(C-)"
- note removed: "PU3-OC(C+)"
- note removed: "PU4"
- note removed: "PU4-IC(C-)"
- note removed: "PU4-OC(C+)"
- note removed: "PWR SWITCH"
- note removed: "STRING GND"
- note removed: "VBATT"
- note removed: "VCC(+)"
- note removed: "v1.2"
