File: XR_Preamp/XR_Preamp.sch (EAGLE design)
At the start: 10 parts, among them U1 XR_PREAMP

Commit message: Updated BOM and Document Number
Parts:
- removed H1: (no value), con-lstb:MA07-2
- removed PAD6, PAD7: (no value), wirepad:SMD2
- removed TR1: TC33X-2-201E, CYCFI_Passive:TC33X-2-201E
- removed U1: XR_PREAMP, CYCFI_Module_castellated:XR_PREAMP
- added C1, C3: 4.7uF, resistor:C-EUC0603
- added C2: 100pF, resistor:C-EUC0402
- added C4: 0.1uf, resistor:C-EUC0402
- added C5: 4.7uF, resistor:C-EUC0402
- added R1: 200K, resistor:R-EU_R0402
- added R2: 27K, resistor:R-EU_R0402
- added R3: 22K, resistor:R-EU_R0402
- added R4, R5: 10K, resistor:R-EU_R0402
- added R6: 4.7K, resistor:R-EU_R0402
- added R7: 1K, resistor:R-EU_R0402
- added T1, T2: 2SC3324, transistor:BC846
- PAD1, PAD2, PAD3, PAD4, PAD5: value (none) -> WIREPAD2,15/1,0; device wirepad:SMD2 -> wirepad:1,6/0,8
Connections:
- removed net INPUT: H1.5, U1.IN
- removed net OUT(PREAMP): H1.8, U1.OUT
- removed net OUT(SEL): H1.10, PAD2.P
- removed net OUT(VOL): H1.1, H1.4, PAD3.P
- removed net SW: H1.2, H1.9
- new net GAIN: PAD1.P, R7.2, T1.E
- new net IN: C1.1, C2.2, PAD3.P
- new net N$3: C5.2, R4.2, T2.E
- new net OUT: PAD5.P, R6.2
- new net OUT1: C5.1, R5.2, R6.1
- new net VCVF: R1.2, R3.1, T1.C, T2.B
- net GND: now also C2.1, C3.1, C4.1, PAD2.P, R2.1, R4.1, R5.1, R7.1; no longer H1.13, H1.14, H1.3, H1.6, H1.7, PAD1.P, PAD4.P, PAD5.P, PAD6.P, PAD7.P, TR1.3, U1.GND
- net N$1: now also C1.2, R1.1, R2.2, T1.B; no longer TR1.2, U1.GAIN
- net VCC: now also C3.2, C4.2, PAD4.P, R3.2, T2.C; no longer H1.11, H1.12, U1.VCC
Other:
- note added: "1/2"
- note added: "2/2"
- note added: "2016008"
- note added: "CASTELLATED PADS"
- note added: "GND"
- note added: "NOTE: *Gain Adjustment Trimmer"
- note added: "TR1 500 0hms"
- note added: "VCC"
- note added: "XR Preamp"
- note added: "XR Preamp for XR Project by Cycfi Research is licensed under a Creative Commons Attribution-ShareAlike 4.0 International License. http://creativecommons.org/licenses/by-sa/4.0/ Copyright CYCFI Research Inc. 2013-2017"
- note added: "v1.5"
- note removed: "-(SW)"
- note removed: "2016039"
- note removed: "500 ohms"
- note removed: "Active Volume"
- note removed: "Active Volume Project by Cycfi Research is licensed under a Creative Commons Attribution-ShareAlike 4.0 International License. http://creativecommons.org/licenses/by-sa/4.0/ Copyright CYCFI Research Inc. 2013-2017"
- note removed: "COIL"
- note removed: "GND(-)"
- note removed: "IN"
- note removed: "INSERT"
- note removed: "NOTES: *POTENTIOMETER BREAKOUT = SMD pads for potentiometer breakout board (POT1)"
- note removed: "OUT"
- note removed: "OUTPUT HEADERS"
- note removed: "OUTPUT JACK"
- note removed: "OUT\"
- note removed: "POT1 25K"
- note removed: "POTENTIOMETER BREAKOUT"
- note removed: "PWR"
- note removed: "SW"
- note removed: "TONE CONTROL"
- note removed: "VCC(+)"
- note removed: "v1.1"
